File: ECAD/OpenTallyESP32/OpenTallyESP32.kicad_sch (KiCad schematic)
At the start: 1 part, among them U1 XIAO ESP32C3

Commit message: Added ESP32
Parts:
- added D1, D2: WS2812B, LED_SMD:LED_WS2812B_PLCC4_5.0x5.0mm_P3.2mm, symbol LED:WS2812B
- added R1, R2: R_Small, symbol Device:R_Small
- added U2: ESP32-C3-WROOM-02, RF_Module:ESP32-C3-WROOM-02, symbol RF_Module:ESP32-C3-WROOM-02
Connections:
- net BATT_LEVEL: now reaches U1.1 (D0)
- net BATT_LEVEL: now also R1.2, R2.1
- net +3.3V: now reaches U1.12 (VCC_3V3)
- net +3.3V: now also D1.1 (VDD), D2.1 (VDD)
- net GND: now reaches U1.13 (GND)
- net GND: now also D1.3 (VSS), D2.3 (VSS)
- net NEOPIXEL: now reaches U1.9 (D8)
- net NEOPIXEL: now also D2.4 (DIN)
- net +BATT: now reaches U1.B+ (Batt+)
- net +BATT: now also R1.1
- net -BATT: now reaches U1.B- (Batt-)
- net -BATT: now also R2.2
- new net: D1.4 (DIN), D2.2 (DOUT)
- new net: U2.19 (GND), U2.9 (GND)
- no-connect marks 0 -> 1
Other:
- moved on the sheet: U1

Commit message: Jeff a terminé la chignole
Parts:
- removed U2: ESP32-C3-WROOM-02, RF_Module:ESP32-C3-WROOM-02, symbol RF_Module:ESP32-C3-WROOM-02
- added C1, C2: C_Small, Capacitor_SMD:C_1206_3216Metric_Pad1.33x1.80mm_HandSolder, symbol Device:C_Small
- added J1: Conn_01x02, Resistor_SMD:R_2512_6332Metric_Pad1.40x3.35mm_HandSolder, symbol Connector_Generic:Conn_01x02
- added Q1: AO3400A, Package_TO_SOT_SMD:SOT-23, symbol Transistor_FET:AO3400A
- added R3: R_Small, Resistor_SMD:R_1206_3216Metric_Pad1.30x1.75mm_HandSolder, symbol Device:R_Small
- added SW1: SW_Push, Button_Switch_SMD:SW_Push_1P1T_NO_CK_KMR2, symbol Switch:SW_Push
- R1, R2: footprint (none) -> Resistor_SMD:R_1206_3216Metric_Pad1.30x1.75mm_HandSolder
Connections:
- net +3.3V: now also C1.1, C2.1
- net +BATT: now also U1.15 (Batt+), J1.2 (Pin_2); no longer U1.B+ (Batt+)
- net -BATT: now also U1.16 (Batt-), J1.1 (Pin_1), Q1.2 (S); no longer R2.2, U1.B- (Batt-)
- net BATT_LEVEL: now also U1.3 (D2); no longer U1.1 (D0)
- net GND: now also C1.2, C2.2, SW1.2
- net SW: now reaches U1.2 (D1)
- net SW: now also SW1.1
- new net: Q1.3 (D), R2.2
- new net: Q1.1 (G), R3.2
- new net BATT_READ: R3.1, U1.1 (D0)
Other:
- moved on the sheet: D1, D2, R1, R2
